Commit message: Update radar.xacro

File: description/radar.xacro (robot description, xacro)
@@ -1,10 +1,10 @@
 <?xml version="1.0"?>
 <robot xmlns:xacro="http://www.ros.org/wiki/xacro" >
-    <joint name="laser_joint1" type="fixed">
+    <joint name="radar_joint" type="fixed">
         <parent link="chassis"/>
-        <child link="laser_frame1"/>
+        <child link="radar_frame"/>
         <origin xyz="0.1 0 0.175" rpy="0 0 0"/>
     </joint>
-    <link name="laser_frame1">
+    <link name="radar_frame">
         <visual>
             <geometry>
@@ -19,10 +19,10 @@
         </collision>
         <xacro:inertial_cylinder mass="0.1" length="0.04" radius="0.05">
-            <origin xyz="0 0 0" rpy="0 0 0"/>
+            <origin xyz="0 0 0"  rpy="0 0 0"/>
         </xacro:inertial_cylinder>
     </link>
-    <gazebo reference="laser_frame1">
+    <gazebo reference="radar_frame">
         <material>Gazebo/Orange</material>
-        <sensor name="laser" type="ray">
+        <sensor name="radar" type="ray">
             <pose> 0 0 0 0 0 0 </pose>
             <visualize>true</visualize>
@@ -35,4 +35,9 @@
                         <max_angle>0.65</max_angle>
                     </horizontal>
+                 <!--   <vertical>
+                        <samples>130</samples>
+                        <min_angle>-0.2</min_angle>
+                        <max_angle>0.2</max_angle>
+                    </vertical> -->
                 </scan>
                 <range>
@@ -41,10 +46,15 @@
                 </range>
             </ray>
-            <plugin name="laser_controller1" filename="libgazebo_ros_ray_sensor.so">
+            <plugin name="radar_controller" filename="libgazebo_ros_ray_sensor.so">
                 <ros>
                     <argument>~/out:=scan</argument>
                 </ros>
                 <output_type>sensor_msgs/LaserScan</output_type>
-                <frame_name>laser_frame1</frame_name>
+                <frame_name>radar_frame</frame_name>
+                <recording>
+                    <enable>true</enable>
+                    <filename>/sep_bot/src/sep_bot/send/output.pcap</filename>
+                    <format>pcap</format>
+                </recording>
             </plugin>
         </sensor>
